Commit message: update content

File: day1/iai_kitchen/urdf_obj/IAI_tables.urdf.xacro (robot description, xacro)
@@ -27,5 +27,5 @@
       <xacro:sphere_inertia radius="0" mass="0"/>
       <visual>
-        <origin xyz="0.0 0.0 0.0" rpy="0 0 0" />
+        <origin xyz="0.0 0.0 0.4" rpy="0 0 0" />
         <geometry>
           <mesh filename="package://iai_kitchen/meshes/jokkmokk/JokkmokkTable.dae"/>

File: day1/kitchen.urdf.xacro (robot description, xacro)
@@ -6,8 +6,6 @@
     <xacro:include filename="$(find iai_kitchen)/urdf_obj/IAI_fridge_area.urdf.xacro" />
     <xacro:include filename="$(find iai_kitchen)/urdf_obj/IAI_tables.urdf.xacro" />
-    <xacro:include filename="$(find iai_kitchen)/urdf_obj/IAI_kitchen_walls.urdf.xacro" />
     <xacro:property name="pi" value="3.1415926535897931" />
     <xacro:property name="simulated" value="true" />
-    <xacro:property name="include_wall_7" value="false" />
     <xacro:macro name="sphere_inertia" params="radius mass">
         <inertial>
@@ -31,24 +29,16 @@
         </joint>
     </xacro:if>
-    <xacro:iai_sink_area name="sink_area" parent="room_link">
-        <origin xyz="1.855 1.3 0" rpy="0 0 ${pi}" />
-    </xacro:iai_sink_area>
-    <xacro:iai_oven_area name="oven_area" parent="room_link">
-        <origin xyz="1.845 2.5 0" rpy="0 0 ${pi}" />
-    </xacro:iai_oven_area>
-    <xacro:iai_kitchen_island name="kitchen_island" parent="room_link">
-        <origin xyz="-1.363 0.59 0" rpy="0 0 0" />
-    </xacro:iai_kitchen_island>
-    <xacro:iai_fridge_area name="fridge_area" parent="room_link">
-        <origin xyz="1.845 -0.73 0" rpy="0 0 ${pi}" />
+    <!-- Your code goes from here -->
+    <!-- fridge -->
+    <xacro:iai_fridge_area name="fridge_1" parent="room_link">
+        <origin xyz="0 0 0" rpy="0 0 ${pi}" />
     </xacro:iai_fridge_area>
-    <xacro:iai_table_1 name="table_area" parent="room_link">
-        <origin xyz="-2.4 -1.5 0" rpy="0 0 ${pi}" />
-    </xacro:iai_table_1>
-    <xacro:iai_dining_area name="dining_area" parent="room_link">
-        <origin xyz="-3.38 0.28 0" rpy="0 0 ${pi / 2}" />
-    </xacro:iai_dining_area>
-    <xacro:iai_kitchen_wall_robohow parent="room_link">
-        <origin xyz="-0.96 0.65 0" rpy="0.0 0.0 0.0" />
-    </xacro:iai_kitchen_wall_robohow>
+    <!-- Dishwasher -->
+    <xacro:iai_dish_washer name="dishwaser_1" parent="room_link">
+        <origin xyz="-0.3 -1 0.4" rpy="0 0 ${pi}" />
+    </xacro:iai_dish_washer>
+    <!-- Oven -->
+    <xacro:iai_oven name="oven_1" parent="room_link">
+        <origin xyz="-0.3 0.4 0.4" rpy="0 0 ${pi}" />
+    </xacro:iai_oven>
 </robot>

Commit message: update extension, fix kitchen urdf errors

File: day1/iai_kitchen/urdf_obj/IAI_tables.urdf.xacro (robot description, xacro)
@@ -33,5 +33,5 @@
       </visual>
       <collision>
-        <origin xyz="0.0 0.0 0.0" rpy="0 0 0" />
+        <origin xyz="0.0 0.0 0.4" rpy="0 0 0" />
         <geometry>
           <mesh filename="package://iai_kitchen/meshes/jokkmokk/JokkmokkTable.obj"/>
